File: switch.kicad_sch (KiCad schematic)
At the start: 13 parts, among them Q1 NTR4003N, Q2 NTR4003N, Q3 DMG2305UX

Commit message: Fixed models and simulation
Parts:
- removed D1: SS24, symbol Device:D_Schottky_Filled
- added D2: SS24, symbol Device:D_Schottky_Filled
- renumbered D2 to D1, R7 to R1, R9 to R2, R8 to R3, R10 to R4, R6 to R5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
Connections:
- net LOAD: now also D2.1 (K)
- net VBUS: now also D2.2 (A)
